File: ArduSatMultipleProcessorModule.sch (EAGLE design)
At the start: 86 parts, among them IC1 ATMEGA328P, IC2 ATMEGA328P, IC3 ATMEGA328P, IC4 ATMEGA328P, IC7 ATMEGA328P, IC8 MCP23S17ML, P1 N1_ICSP, P2 N0_ICSP, P3 N0_ICSP, P4 N1_ICSP, P5 N1_ICSP, Q1 BSS138 N-MOSFET, Q10 2N7002 N-MOSFET, Q11 BSS138 N-MOSFET, Q12 BSS138 N-MOSFET, Q2 BSS138 N-MOSFET, Q3 BSS138 N-MOSFET, Q4 BSS138 N-MOSFET, Q5 BSS138 N-MOSFET, Q6 BSS138 N-MOSFET, Q7 BSS138 N-MOSFET, Q8 BSS138 N-MOSFET, Q9 2N7002 N-MOSFET

Commit message: Experiments in node dimensions and layout
Parts:
- P4: device freetronics-jon:ICSPSMT -> freetronics-jon:ICSPPTH
Connections:
- net +5V_SYS: now also Q11.G, Q12.G, R22.2, R23.2
- net GND: now also RN3A.1; no longer RN3B.1
- net N$19: now also U$38.C-G; no longer U$38.C-R
- net N$20: now also RN3B.2, U$38.C-R; no longer RN3D.2, U$38.C-G
- net N$21: now also RN3A.2; no longer RN3B.2
- net N1_5V: no longer Q11.G, Q12.G, R22.2, R23.2
- net N1_D0_RX: now also RN3C.1; no longer RN3D.1
- net N1_D1_TX: now also RN3B.1; no longer RN3C.1
Other:
- moved on the sheet: RN3A, RN3B, RN3C, RN3D
Changed lines of the file:
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@@
 <part name="R16" library="freetronics-master-v1.1" deviceset="RESISTOR" device="0603" value="22K 0603"/>
 <part name="U$35" library="SparkFun" deviceset="5V" device=""/>
-<part name="P4" library="freetronics-jon" deviceset="ICSP" device="SMT" value="N1_ICSP"/>
+<part name="P4" library="freetronics-jon" deviceset="ICSP" device="PTH" value="N1_ICSP"/>
 <part name="GND19" library="SparkFun" deviceset="GND" device=""/>
 <part name="U$36" library="SparkFun" deviceset="5V" device=""/>
@@
 <instance part="U$37" gate="G$1" x="147.32" y="238.76" rot="R270"/>
 <instance part="U$38" gate="G$1" x="86.36" y="266.7" rot="R180"/>
-<instance part="RN3" gate="A" x="99.06" y="251.46" rot="R180"/>
-<instance part="RN3" gate="B" x="99.06" y="259.08" rot="R180"/>
-<instance part="RN3" gate="C" x="99.06" y="266.7" rot="R180"/>
-<instance part="RN3" gate="D" x="99.06" y="274.32" rot="R180"/>
+<instance part="RN3" gate="A" x="99.06" y="259.08" rot="R180"/>
+<instance part="RN3" gate="B" x="99.06" y="266.7" rot="R180"/>
+<instance part="RN3" gate="C" x="99.06" y="274.32" rot="R180"/>
+<instance part="RN3" gate="D" x="99.06" y="279.4" rot="R180"/>
 <instance part="U$39" gate="G$1" x="58.42" y="266.7"/>
-<instance part="GND20" gate="1" x="106.68" y="256.54"/>
+<instance part="GND20" gate="1" x="109.22" y="256.54"/>
 <instance part="U$40" gate="G$1" x="154.94" y="251.46"/>
 <instance part="GND21" gate="1" x="170.18" y="215.9"/>
@@
 <label x="165.1" y="157.48" size="1.778" layer="95" rot="R90"/>
 </segment>
+<segment>
+<pinref part="Q11" gate="G$1" pin="G"/>
+<pinref part="U$45" gate="G$1" pin="5V"/>
+<wire x1="302.26" y1="50.8" x2="302.26" y2="55.88" width="0.1524" layer="91"/>
+<pinref part="R22" gate="G$1" pin="2"/>
+<wire x1="302.26" y1="55.88" x2="304.8" y2="55.88" width="0.1524" layer="91"/>
+<wire x1="284.48" y1="53.34" x2="284.48" y2="55.88" width="0.1524" layer="91"/>
+<wire x1="284.48" y1="55.88" x2="302.26" y2="55.88" width="0.1524" layer="91"/>
+<junction x="302.26" y="55.88"/>
+<label x="287.02" y="55.88" size="1.778" layer="95"/>
+</segment>
+<segment>
+<pinref part="Q12" gate="G$1" pin="G"/>
+<pinref part="U$46" gate="G$1" pin="5V"/>
+<wire x1="302.26" y1="25.4" x2="302.26" y2="30.48" width="0.1524" layer="91"/>
+<pinref part="R23" gate="G$1" pin="2"/>
+<wire x1="302.26" y1="30.48" x2="304.8" y2="30.48" width="0.1524" layer="91"/>
+<wire x1="284.48" y1="27.94" x2="284.48" y2="30.48" width="0.1524" layer="91"/>
+<wire x1="284.48" y1="30.48" x2="302.26" y2="30.48" width="0.1524" layer="91"/>
+<junction x="302.26" y="30.48"/>
+<label x="287.02" y="30.48" size="1.778" layer="95"/>
+</segment>
 </net>
 <net name="VCC_SYS" class="0">
@@
 </segment>
 <segment>
-<pinref part="RN3" gate="B" pin="1"/>
-<wire x1="104.14" y1="259.08" x2="106.68" y2="259.08" width="0.1524" layer="91"/>
-<pinref part="GND20" gate="1" pin="GND"/>
-</segment>
-<segment>
 <wire x1="271.78" y1="139.7" x2="266.7" y2="139.7" width="0.1524" layer="91"/>
 <wire x1="266.7" y1="139.7" x2="266.7" y2="134.62" width="0.1524" layer="91"/>
@@
 <junction x="429.26" y="20.32"/>
 </segment>
+<segment>
+<pinref part="RN3" gate="A" pin="1"/>
+<pinref part="GND20" gate="1" pin="GND"/>
+<wire x1="109.22" y1="259.08" x2="104.14" y2="259.08" width="0.1524" layer="91"/>
+</segment>
 </net>
 <net name="AGND" class="0">
@@
 <wire x1="30.48" y1="261.62" x2="43.18" y2="261.62" width="0.1524" layer="91"/>
 </segment>
-<segment>
-<pinref part="Q12" gate="G$1" pin="G"/>
-<pinref part="U$46" gate="G$1" pin="5V"/>
-<wire x1="302.26" y1="25.4" x2="302.26" y2="30.48" width="0.1524" layer="91"/>
-<pinref part="R23" gate="G$1" pin="2"/>
-<wire x1="302.26" y1="30.48" x2="304.8" y2="30.48" width="0.1524" layer="91"/>
-<wire x1="284.48" y1="27.94" x2="284.48" y2="30.48" width="0.1524" layer="91"/>
-<wire x1="284.48" y1="30.48" x2="302.26" y2="30.48" width="0.1524" layer="91"/>
-<junction x="302.26" y="30.48"/>
-<label x="287.02" y="30.48" size="1.778" layer="95"/>
-</segment>
-<segment>
-<pinref part="Q11" gate="G$1" pin="G"/>
-<pinref part="U$45" gate="G$1" pin="5V"/>
-<wire x1="302.26" y1="50.8" x2="302.26" y2="55.88" width="0.1524" layer="91"/>
-<pinref part="R22" gate="G$1" pin="2"/>
-<wire x1="302.26" y1="55.88" x2="304.8" y2="55.88" width="0.1524" layer="91"/>
-<wire x1="284.48" y1="53.34" x2="284.48" y2="55.88" width="0.1524" layer="91"/>
-<wire x1="284.48" y1="55.88" x2="302.26" y2="55.88" width="0.1524" layer="91"/>
-<junction x="302.26" y="55.88"/>
-<label x="287.02" y="55.88" size="1.778" layer="95"/>
-</segment>
 </net>
 <net name="N1_D13_SCK" class="0">
@@
 <net name="N1_D0_RX" class="0">
 <segment>
-<pinref part="RN3" gate="D" pin="1"/>
 <label x="106.68" y="274.32" size="1.778" layer="95"/>
 <wire x1="104.14" y1="274.32" x2="119.38" y2="274.32" width="0.1524" layer="91"/>
+<pinref part="RN3" gate="C" pin="1"/>
 </segment>
 <segment>
@@
 <net name="N1_D1_TX" class="0">
 <segment>
-<pinref part="RN3" gate="C" pin="1"/>
 <label x="106.68" y="266.7" size="1.778" layer="95"/>
 <wire x1="104.14" y1="266.7" x2="119.38" y2="266.7" width="0.1524" layer="91"/>
+<pinref part="RN3" gate="B" pin="1"/>
 </segment>
 <segment>
@@
 </segment>
 </net>
-<net name="N$19" class="0">
-<segment>
-<pinref part="U$38" gate="G$1" pin="C-R"/>
-<pinref part="RN3" gate="C" pin="2"/>
-</segment>
-</net>
-<net name="N$20" class="0">
-<segment>
-<pinref part="U$38" gate="G$1" pin="C-G"/>
-<pinref part="RN3" gate="D" pin="2"/>
-</segment>
-</net>
-<net name="N$21" class="0">
-<segment>
-<pinref part="U$38" gate="G$1" pin="C-B"/>
-<pinref part="RN3" gate="B" pin="2"/>
-</segment>
-</net>
 <net name="N2_5V" class="0">
 <segment>
@@
 </segment>
 </net>
+<net name="N$21" class="0">
+<segment>
+<pinref part="U$38" gate="G$1" pin="C-B"/>
+<pinref part="RN3" gate="A" pin="2"/>
+</segment>
+</net>
+<net name="N$19" class="0">
+<segment>
+<pinref part="U$38" gate="G$1" pin="C-G"/>
+<pinref part="RN3" gate="C" pin="2"/>
+</segment>
+</net>
+<net name="N$20" class="0">
+<segment>
+<pinref part="U$38" gate="G$1" pin="C-R"/>
+<pinref part="RN3" gate="B" pin="2"/>
+</segment>
+</net>

Commit message: Added parts for remaining nodes
Parts:
- added C12, C21, C24, C25, C26, C33, C36, C37, C38, C45, C48, C49, C50: 100nF 0603, freetronics-master-v1.1:CAP0603
- added C16, C17, C18, C19, C20, C22, C23, C27, C28, C29, C30, C31, C32, C34, C35, C39, C40, C41, C42, C43, C44, C46, C47: 22pF 0603, freetronics-master-v1.1:CAP0603
- added IC10, IC11, IC12, IC13, IC14, IC15, IC16, IC17, IC18, IC5, IC6, IC9: ATMEGA328P, freetronics-master-v1.1:AVR-MEGA8-MI
- added P10, P12, P14, P16, P6, P8: N0_ICSP, freetronics-jon:ICSPPTH
- added P11, P13, P15, P17, P7, P9: N1_ICSP, freetronics-jon:ICSPPTH
- added Q13, Q14, Q23, Q24, Q25, Q26, Q35, Q36, Q37, Q38, Q47, Q48, Q49, Q50: 2N7002 N-MOSFET, freetronics-master-v1:MOSFET-NCHANNELSMD
- added Q15, Q16, Q17, Q18, Q19, Q20, Q21, Q22, Q27, Q28, Q29, Q30, Q31, Q32, Q33, Q34, Q39, Q40, Q41, Q42, Q43, Q44, Q45, Q46: BSS138 N-MOSFET, freetronics-master-v1:MOSFET-NCHANNELSMD
- added R24, R29, R35, R39, R43, R47, R51, R55, R59, R63, R67, R71: 22K 0603, freetronics-master-v1.1:RESISTOR0603
- added R25, R30, R36, R40, R44, R48, R52, R56, R60, R64, R68, R72: 1M 0603, freetronics-master-v1.1:RESISTOR0603
- added R27, R28, R31, R34, R37, R38, R41, R42, R45, R46, R49, R50, R53, R54, R57, R58, R61, R62, R65, R66, R69, R70, R73, R74: 10K 0603, freetronics-master-v1.1:RESISTOR0603
- added RN10, RN11, RN12, RN13, RN14, RN15, RN16, RN5, RN6, RN7, RN8, RN9: 2K2, resistor-dil:4R-NCAY16
- added U$106, U$114, U$124, U$132, U$140, U$148, U$48, U$64, U$72, U$80, U$90, U$98: CRYSTAL-GND3X2, freetronics-jon:CRYSTAL-GND3X2
- added U$107, U$115, U$125, U$133, U$141, U$149, U$49, U$65, U$73, U$81, U$91, U$99: RGBLEDSMT, freetronics-jon:RGBLEDSMT
- C6: value 100nF 0603 -> 22pF 0603
- P1, P2: device freetronics-jon:ICSPSMT -> freetronics-jon:ICSPPTH
Connections:
- new net N$113: C18.2, IC6.PB7(XTAL2/TOSC2), R30.1, U$64.XTL2
- new net N$114: C17.2, IC6.PB6(XTAL1/TOSC1), R30.2, U$64.XTL1
- new net N$115: RN6C.2, U$65.C-G
- new net N$117: RN6B.2, U$65.C-R
- new net N$126: RN6A.2, U$65.C-B
- new net N$182: C20.2, IC9.PB7(XTAL2/TOSC2), R36.1, U$72.XTL2
- new net N$192: C19.2, IC9.PB6(XTAL1/TOSC1), R36.2, U$72.XTL1
- new net N$193: C23.2, IC10.PB7(XTAL2/TOSC2), R40.1, U$80.XTL2
- new net N$194: C22.2, IC10.PB6(XTAL1/TOSC1), R40.2, U$80.XTL1
- new net N$195: RN8A.2, U$81.C-B
- new net N$196: RN8C.2, U$81.C-G
- new net N$201: RN8B.2, U$81.C-R
- new net N$202: RN7B.2, U$73.C-R
- new net N$214: RN7C.2, U$73.C-G
- new net N$220: RN7A.2, U$73.C-B
- new net N$226: C28.2, IC11.PB7(XTAL2/TOSC2), R44.1, U$90.XTL2
- new net N$232: C27.2, IC11.PB6(XTAL1/TOSC1), R44.2, U$90.XTL1
- new net N$233: C30.2, IC12.PB7(XTAL2/TOSC2), R48.1, U$98.XTL2
- new net N$234: C29.2, IC12.PB6(XTAL1/TOSC1), R48.2, U$98.XTL1
- new net N$235: C32.2, IC13.PB7(XTAL2/TOSC2), R52.1, U$106.XTL2
- new net N$24: C16.2, IC5.PB7(XTAL2/TOSC2), R25.1, U$48.XTL2
- new net N$248: C31.2, IC13.PB6(XTAL1/TOSC1), R52.2, U$106.XTL1
- new net N$249: C35.2, IC14.PB7(XTAL2/TOSC2), R56.1, U$114.XTL2
- new net N$250: C34.2, IC14.PB6(XTAL1/TOSC1), R56.2, U$114.XTL1
- new net N$251: RN12A.2, U$115.C-B
- new net N$252: RN12C.2, U$115.C-G
- new net N$255: RN12B.2, U$115.C-R
- new net N$26: C6.2, IC5.PB6(XTAL1/TOSC1), R25.2, U$48.XTL1
- new net N$299: RN11B.2, U$107.C-R
- new net N$310: RN11C.2, U$107.C-G
- new net N$311: RN11A.2, U$107.C-B
- new net N$321: C40.2, IC15.PB7(XTAL2/TOSC2), R60.1, U$124.XTL2
- new net N$338: C39.2, IC15.PB6(XTAL1/TOSC1), R60.2, U$124.XTL1
- new net N$356: C42.2, IC16.PB7(XTAL2/TOSC2), R64.1, U$132.XTL2
- new net N$367: C41.2, IC16.PB6(XTAL1/TOSC1), R64.2, U$132.XTL1
- new net N$374: C44.2, IC17.PB7(XTAL2/TOSC2), R68.1, U$140.XTL2
- new net N$378: C43.2, IC17.PB6(XTAL1/TOSC1), R68.2, U$140.XTL1
- new net N$384: C47.2, IC18.PB7(XTAL2/TOSC2), R72.1, U$148.XTL2
- new net N$39: RN5C.2, U$49.C-G
- new net N$41: RN5B.2, U$49.C-R
- new net N$416: C46.2, IC18.PB6(XTAL1/TOSC1), R72.2, U$148.XTL1
- new net N$417: RN16A.2, U$149.C-B
- new net N$418: RN16C.2, U$149.C-G
- new net N$419: RN16B.2, U$149.C-R
- new net N$42: RN5A.2, U$49.C-B
- new net N$420: RN15B.2, U$141.C-R
- new net N$421: RN15C.2, U$141.C-G
- new net N$422: RN15A.2, U$141.C-B
- new net N$423: RN9C.2, U$91.C-G
- new net N$424: RN9B.2, U$91.C-R
- new net N$425: RN9A.2, U$91.C-B
- new net N$426: RN10C.2, U$99.C-G
- new net N$427: RN10B.2, U$99.C-R
- new net N$428: RN10A.2, U$99.C-B
- new net N$429: RN13C.2, U$125.C-G
- new net N$430: RN13B.2, U$125.C-R
- new net N$431: RN13A.2, U$125.C-B
- new net N$432: RN14C.2, U$133.C-G
- new net N$433: RN14B.2, U$133.C-R
- new net N$434: RN14A.2, U$133.C-B
- new net N10_5V: C37.1, IC11.AREF, IC11.AVCC, IC11.VCC@1, IC11.VCC@2, P10.2, Q27.G, Q28.G, Q37.D, R43.2, R45.2, R46.2, U$91.A-G, U$91.A-R
- new net N10_A4_SDA: IC11.PC4(ADC4/SDA), Q27.S, R45.1
- new net N10_A5_SCL: IC11.PC5(ADC5/SCL), Q28.S, R46.1
- new net N10_D11_MOSI: IC11.PB3(MOSI/OC2), P10.4
- new net N10_D12_MISO: IC11.PB4(MISO), P10.1
- new net N10_D13_SCK: IC11.PB5(SCK), P10.3, U$91.A-B
- new net N10_RESET: IC11.PC6(/RESET), P10.5, R43.1
- new net N11_5V: C38.1, IC12.AREF, IC12.AVCC, IC12.VCC@1, IC12.VCC@2, P11.2, Q29.G, Q30.G, Q38.D, R47.2, R49.2, R50.2, U$99.A-G, U$99.A-R
- new net N11_A4_SDA: IC12.PC4(ADC4/SDA), Q29.S, R49.1
- new net N11_A5_SCL: IC12.PC5(ADC5/SCL), Q30.S, R50.1
- new net N11_D11_MOSI: IC12.PB3(MOSI/OC2), P11.4
- new net N11_D12_MISO: IC12.PB4(MISO), P11.1
- new net N11_D13_SCK: IC12.PB5(SCK), P11.3, U$99.A-B
- new net N11_RESET: IC12.PC6(/RESET), P11.5, R47.1
- new net N12_5V: C45.1, IC17.AREF, IC17.AVCC, IC17.VCC@1, IC17.VCC@2, P16.2, Q43.G, Q44.G, Q47.D, R67.2, R69.2, R70.2, U$141.A-G, U$141.A-R
- new net N12_A4_SDA: IC17.PC4(ADC4/SDA), Q43.S, R69.1
- new net N12_A5_SCL: IC17.PC5(ADC5/SCL), Q44.S, R70.1
- new net N12_D11_MOSI: IC17.PB3(MOSI/OC2), P16.4
- new net N12_D12_MISO: IC17.PB4(MISO), P16.1
- new net N12_D13_SCK: IC17.PB5(SCK), P16.3, U$141.A-B
- new net N12_RESET: IC17.PC6(/RESET), P16.5, R67.1
- new net N13_5V: C48.1, IC18.AREF, IC18.AVCC, IC18.VCC@1, IC18.VCC@2, P17.2, Q45.G, Q46.G, Q48.D, R71.2, R73.2, R74.2, U$149.A-G, U$149.A-R
- new net N13_A4_SDA: IC18.PC4(ADC4/SDA), Q45.S, R73.1
- new net N13_A5_SCL: IC18.PC5(ADC5/SCL), Q46.S, R74.1
- new net N13_D11_MOSI: IC18.PB3(MOSI/OC2), P17.4
- new net N13_D12_MISO: IC18.PB4(MISO), P17.1
- new net N13_D13_SCK: IC18.PB5(SCK), P17.3, U$149.A-B
- new net N13_RESET: IC18.PC6(/RESET), P17.5, R71.1
- new net N14_5V: C49.1, IC15.AREF, IC15.AVCC, IC15.VCC@1, IC15.VCC@2, P14.2, Q39.G, Q40.G, Q49.D, R59.2, R61.2, R62.2, U$125.A-G, U$125.A-R
- new net N14_A4_SDA: IC15.PC4(ADC4/SDA), Q39.S, R61.1
- new net N14_A5_SCL: IC15.PC5(ADC5/SCL), Q40.S, R62.1
- new net N14_D11_MOSI: IC15.PB3(MOSI/OC2), P14.4
- new net N14_D12_MISO: IC15.PB4(MISO), P14.1
- new net N14_D13_SCK: IC15.PB5(SCK), P14.3
- new net N14_RESET: IC15.PC6(/RESET), P14.5, R59.1
- new net N15_5V: C50.1, IC16.AREF, IC16.AVCC, IC16.VCC@1, IC16.VCC@2, P15.2, Q41.G, Q42.G, Q50.D, R63.2, R65.2, R66.2, U$133.A-G, U$133.A-R
- new net N15_A4_SDA: IC16.PC4(ADC4/SDA), Q41.S, R65.1
- new net N15_A5_SCL: IC16.PC5(ADC5/SCL), Q42.S, R66.1
- new net N15_D11_MOSI: IC16.PB3(MOSI/OC2), P15.4
- new net N15_D12_MISO: IC16.PB4(MISO), P15.1
- new net N15_D13_SCK: IC16.PB5(SCK), P15.3, U$133.A-B
- new net N15_RESET: IC16.PC6(/RESET), P15.5, R63.1
- new net N4_5V: C21.1, IC9.AREF, IC9.AVCC, IC9.VCC@1, IC9.VCC@2, P8.2, Q19.G, Q20.G, Q23.D, R35.2, R37.2, R38.2, U$73.A-G, U$73.A-R
- new net N4_A4_SDA: IC9.PC4(ADC4/SDA), Q19.S, R37.1
- new net N4_A5_SCL: IC9.PC5(ADC5/SCL), Q20.S, R38.1
- new net N4_D11_MOSI: IC9.PB3(MOSI/OC2), P8.4
- new net N4_D12_MISO: IC9.PB4(MISO), P8.1
- new net N4_D13_SCK: IC9.PB5(SCK), P8.3, U$73.A-B
- new net N4_RESET: IC9.PC6(/RESET), P8.5, R35.1
- new net N5_5V: C24.1, IC10.AREF, IC10.AVCC, IC10.VCC@1, IC10.VCC@2, P9.2, Q21.G, Q22.G, Q24.D, R39.2, R41.2, R42.2, U$81.A-G, U$81.A-R
- new net N5_A4_SDA: IC10.PC4(ADC4/SDA), Q21.S, R41.1
- new net N5_A5_SCL: IC10.PC5(ADC5/SCL), Q22.S, R42.1
- new net N5_D11_MOSI: IC10.PB3(MOSI/OC2), P9.4
- new net N5_D12_MISO: IC10.PB4(MISO), P9.1
- new net N5_D13_SCK: IC10.PB5(SCK), P9.3, U$81.A-B
- new net N5_RESET: IC10.PC6(/RESET), P9.5, R39.1
- new net N6_5V: C25.1, IC5.AREF, IC5.AVCC, IC5.VCC@1, IC5.VCC@2, P6.2, Q15.G, Q16.G, Q25.D, R24.2, R27.2, R28.2, U$49.A-G, U$49.A-R
- new net N6_A4_SDA: IC5.PC4(ADC4/SDA), Q15.S, R27.1
- new net N6_A5_SCL: IC5.PC5(ADC5/SCL), Q16.S, R28.1
- new net N6_D11_MOSI: IC5.PB3(MOSI/OC2), P6.4
- new net N6_D12_MISO: IC5.PB4(MISO), P6.1
- new net N6_D13_SCK: IC5.PB5(SCK), P6.3, U$125.A-B, U$49.A-B
- new net N6_RESET: IC5.PC6(/RESET), P6.5, R24.1
- new net N7_5V: C26.1, IC6.AREF, IC6.AVCC, IC6.VCC@1, IC6.VCC@2, P7.2, Q17.G, Q18.G, Q26.D, R29.2, R31.2, R34.2, U$65.A-G, U$65.A-R
- new net N7_A4_SDA: IC6.PC4(ADC4/SDA), Q17.S, R31.1
- new net N7_A5_SCL: IC6.PC5(ADC5/SCL), Q18.S, R34.1
- new net N7_D11_MOSI: IC6.PB3(MOSI/OC2), P7.4
- new net N7_D12_MISO: IC6.PB4(MISO), P7.1
- new net N7_D13_SCK: IC6.PB5(SCK), P7.3, U$65.A-B
- new net N7_RESET: IC6.PC6(/RESET), P7.5, R29.1
- new net N8_5V: C33.1, IC13.AREF, IC13.AVCC, IC13.VCC@1, IC13.VCC@2, P12.2, Q31.G, Q32.G, Q35.D, R51.2, R53.2, R54.2, U$107.A-G, U$107.A-R
- new net N8_A4_SDA: IC13.PC4(ADC4/SDA), Q31.S, R53.1
- new net N8_A5_SCL: IC13.PC5(ADC5/SCL), Q32.S, R54.1
- new net N8_D11_MOSI: IC13.PB3(MOSI/OC2), P12.4
- new net N8_D12_MISO: IC13.PB4(MISO), P12.1
- new net N8_D13_SCK: IC13.PB5(SCK), P12.3, U$107.A-B
- new net N8_RESET: IC13.PC6(/RESET), P12.5, R51.1
- new net N9_5V: C36.1, IC14.AREF, IC14.AVCC, IC14.VCC@1, IC14.VCC@2, P13.2, Q33.G, Q34.G, Q36.D, R55.2, R57.2, R58.2, U$115.A-G, U$115.A-R
- new net N9_A4_SDA: IC14.PC4(ADC4/SDA), Q33.S, R57.1
- new net N9_A5_SCL: IC14.PC5(ADC5/SCL), Q34.S, R58.1
- new net N9_D11_MOSI: IC14.PB3(MOSI/OC2), P13.4
- new net N9_D12_MISO: IC14.PB4(MISO), P13.1
- new net N9_D13_SCK: IC14.PB5(SCK), P13.3, U$115.A-B
- new net N9_RESET: IC14.PC6(/RESET), P13.5, R55.1
- net +5V_SYS: now also Q13.S, Q14.S, Q23.S, Q24.S, Q25.S, Q26.S, Q35.S, Q36.S, Q37.S, Q38.S, Q47.S, Q48.S, Q49.S, Q50.S
- net GND: now also C12.2, C16.1, C17.1, C18.1, C19.1, C20.1, C21.2, C22.1, C23.1, C24.2, C25.2, C26.2, C27.1, C28.1, C29.1, C30.1, C31.1, C32.1, C33.2, C34.1, C35.1, C36.2, C37.2, C38.2, C39.1, C40.1, C41.1, C42.1, C43.1, C44.1, C45.2, C46.1, C47.1, C48.2, C49.2, C50.2, C6.1, IC10.AGND, IC10.GND@1, IC10.GND@2, IC11.AGND, IC11.GND@1, IC11.GND@2, IC12.AGND, IC12.GND@1, IC12.GND@2, IC13.AGND, IC13.GND@1, IC13.GND@2, IC14.AGND, IC14.GND@1, IC14.GND@2, IC15.AGND, IC15.GND@1, IC15.GND@2, IC16.AGND, IC16.GND@1, IC16.GND@2, IC17.AGND, IC17.GND@1, IC17.GND@2, IC18.AGND, IC18.GND@1, IC18.GND@2, IC5.AGND, IC5.GND@1, IC5.GND@2, IC6.AGND, IC6.GND@1, IC6.GND@2, IC9.AGND, IC9.GND@1, IC9.GND@2, P10.6, P11.6, P12.6, P13.6, P14.6, P15.6, P16.6, P17.6, P6.6, P7.6, P8.6, P9.6, RN10A.1, RN11A.1, RN12A.1, RN13A.1, RN14A.1, RN15A.1, RN16A.1, RN1A.1, RN2A.1, RN4A.1, RN5A.1, RN6A.1, RN7A.1, RN8A.1, RN9A.1, U$106.GND, U$106.GND2, U$114.GND, U$114.GND2, U$124.GND, U$124.GND2, U$132.GND, U$132.GND2, U$140.GND, U$140.GND2, U$148.GND, U$148.GND2, U$48.GND, U$48.GND2, U$64.GND, U$64.GND2, U$72.GND, U$72.GND2, U$80.GND, U$80.GND2, U$90.GND, U$90.GND2, U$98.GND, U$98.GND2; no longer C6.2, RN1B.1, RN2B.1, RN4B.1
- net N$10: now also RN1A.2; no longer RN1B.2
- net N$13: now also RN2B.2; no longer RN2C.2
- net N$15: now also RN2C.2; no longer RN2D.2
- net N$16: now also RN2A.2; no longer RN2B.2
- net N$4: now also U$9.C-G; no longer U$9.C-R
- net N$5: now also RN4B.2, U$9.C-R; no longer RN4D.2, U$9.C-G
- net N$6: now also RN4A.2; no longer RN4B.2
- net N$8: now also U$16.C-G; no longer U$16.C-R
- net N$9: now also RN1B.2, U$16.C-R; no longer RN1D.2, U$16.C-G
- net N0_D0_RX: now also RN2C.1; no longer RN2D.1
- net N0_D1_TX: now also RN2B.1; no longer RN2C.1
- net N10_D0_RX: now also IC11.PD0(RXD), RN9C.1
- net N10_D1_TX: now also IC11.PD1(TXD), RN9B.1
- net N10_PWR: now also Q37.G
- net N11_D0_RX: now also IC12.PD0(RXD), RN10C.1
- net N11_D1_TX: now also IC12.PD1(TXD), RN10B.1
- net N11_PWR: now also Q38.G
- net N12_D0_RX: now also IC17.PD0(RXD), RN15C.1
- net N12_D1_TX: now also IC17.PD1(TXD), RN15B.1
- net N12_PWR: now also Q47.G
- net N13_D0_RX: now also IC18.PD0(RXD), RN16C.1
- net N13_D1_TX: now also IC18.PD1(TXD), RN16B.1
- net N13_PWR: now also Q48.G
- net N14_D0_RX: now also IC15.PD0(RXD), RN13C.1
- net N14_D1_TX: now also IC15.PD1(TXD), RN13B.1
- net N14_PWR: now also Q49.G
- net N15_D0_RX: now also IC16.PD0(RXD), RN14C.1
- net N15_D1_TX: now also IC16.PD1(TXD), RN14B.1
- net N15_PWR: now also Q50.G
- net N2_5V: now also C12.1, Q13.D; no longer C4.1
- net N2_D0_RX: now also RN4C.1; no longer RN4D.1
- net N2_D1_TX: now also RN4B.1; no longer RN4C.1
- net N2_PWR: now also Q13.G
- net N3_5V: now also C4.1, Q14.D; no longer C6.1
- net N3_D0_RX: now also RN1C.1; no longer RN1D.1
- net N3_D1_TX: now also RN1B.1; no longer RN1C.1
- net N3_PWR: now also Q14.G
- net N4_D0_RX: now also IC9.PD0(RXD), RN7C.1
- net N4_D1_TX: now also IC9.PD1(TXD), RN7B.1
- net N4_PWR: now also Q23.G
- net N5_D0_RX: now also IC10.PD0(RXD), RN8C.1
- net N5_D1_TX: now also IC10.PD1(TXD), RN8B.1
- net N5_PWR: now also Q24.G
- net N6_D0_RX: now also IC5.PD0(RXD), RN5C.1
- net N6_D1_TX: now also IC5.PD1(TXD), RN5B.1
- net N6_PWR: now also Q25.G
- net N7_D0_RX: now also IC6.PD0(RXD), RN6C.1
- net N7_D1_TX: now also IC6.PD1(TXD), RN6B.1
- net N7_PWR: now also Q26.G
- net N8_D0_RX: now also IC13.PD0(RXD), RN11C.1
- net N8_D1_TX: now also IC13.PD1(TXD), RN11B.1
- net N8_PWR: now also Q35.G
- net N9_D0_RX: now also IC14.PD0(RXD), RN12C.1
- net N9_D1_TX: now also IC14.PD1(TXD), RN12B.1
- net N9_PWR: now also Q36.G
- net NODE_SCL: now also Q16.D, Q18.D, Q20.D, Q22.D, Q28.D, Q30.D, Q32.D, Q34.D, Q40.D, Q42.D, Q44.D, Q46.D
- net NODE_SDA: now also Q15.D, Q17.D, Q19.D, Q21.D, Q27.D, Q29.D, Q31.D, Q33.D, Q39.D, Q41.D, Q43.D, Q45.D
Other:
- note added: "Node 10"
- note added: "Node 11"
- note added: "Node 12"
- note added: "Node 13"
- note added: "Node 14"
- note added: "Node 15"
- note added: "Node 2"
- note added: "Node 3"
- note added: "Node 4"
- note added: "Node 5"
- note added: "Node 6"
- note added: "Node 7"
- note added: "Node 8"
- note added: "Node 9"
- note removed: "Processor Node 2"
- note removed: "Processor Node 3"
- moved on the sheet: C1, C10, C11, C13, C14, C15, C2, C3, C4, C5, C6, C7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
