File: ArduSatMultipleProcessorModule.sch (EAGLE design)
At the start: 268 parts, among them IC1 ATMEGA328P, IC10 ATMEGA328P, IC11 ATMEGA328P, IC12 ATMEGA328P, IC13 ATMEGA328P, IC14 ATMEGA328P, IC15 ATMEGA328P, IC16 ATMEGA328P, IC17 ATMEGA328P, IC18 ATMEGA328P, IC2 ATMEGA328P, IC3 ATMEGA328P, IC4 ATMEGA328P, IC5 ATMEGA328P, IC6 ATMEGA328P, IC7 ATMEGA328P, IC8 MCP23S17ML, IC9 ATMEGA328P, P1 N1_ICSP, P10 N0_ICSP, P11 N1_ICSP, P12 N0_ICSP, P13 N1_ICSP, P14 N0_ICSP, P15 N1_ICSP, P16 N0_ICSP, P17 N1_ICSP, P2 N0_ICSP, P3 N0_ICSP, P4 N1_ICSP, P5 N1_ICSP, P6 N0_ICSP, P7 N1_ICSP, P8 N0_ICSP, P9 N1_ICSP, Q1 BSS138 N-MOSFET, Q10 2N7002 N-MOSFET, Q11 BSS138 N-MOSFET, Q12 BSS138 N-MOSFET, Q13 2N7002 N-MOSFET, Q14 2N7002 N-MOSFET, Q15 BSS138 N-MOSFET, Q16 BSS138 N-MOSFET, Q17 BSS138 N-MOSFET, Q18 BSS138 N-MOSFET, Q19 BSS138 N-MOSFET, Q2 BSS138 N-MOSFET, Q20 BSS138 N-MOSFET, Q21 BSS138 N-MOSFET, Q22 BSS138 N-MOSFET, Q23 2N7002 N-MOSFET, Q24 2N7002 N-MOSFET, Q25 2N7002 N-MOSFET, Q26 2N7002 N-MOSFET, Q27 BSS138 N-MOSFET, Q28 BSS138 N-MOSFET, Q29 BSS138 N-MOSFET, Q3 BSS138 N-MOSFET, Q30 BSS138 N-MOSFET, Q31 BSS138 N-MOSFET, Q32 BSS138 N-MOSFET, Q33 BSS138 N-MOSFET, Q34 BSS138 N-MOSFET, Q35 2N7002 N-MOSFET, Q36 2N7002 N-MOSFET, Q37 2N7002 N-MOSFET, Q38 2N7002 N-MOSFET, Q39 BSS138 N-MOSFET, Q4 BSS138 N-MOSFET, Q40 BSS138 N-MOSFET, Q41 BSS138 N-MOSFET, Q42 BSS138 N-MOSFET, Q43 BSS138 N-MOSFET, Q44 BSS138 N-MOSFET, Q45 BSS138 N-MOSFET, Q46 BSS138 N-MOSFET, Q47 2N7002 N-MOSFET, Q48 2N7002 N-MOSFET, Q49 2N7002 N-MOSFET, Q5 BSS138 N-MOSFET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

Commit message: Routing processor nodes
Connections:
- net N14_D13_SCK: now also U$125.A-B
- net N6_D13_SCK: no longer U$125.A-B
Changed lines of the file:
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@@
 <instance part="RN2" gate="D" x="99.06" y="749.3" rot="R180"/>
 <instance part="U$30" gate="G$1" x="58.42" y="736.6"/>
-<instance part="GND15" gate="1" x="106.68" y="726.44"/>
+<instance part="GND15" gate="1" x="109.22" y="726.44"/>
 <instance part="U$31" gate="G$1" x="154.94" y="721.36"/>
 <instance part="GND16" gate="1" x="170.18" y="685.8"/>
@@
 <pinref part="GND15" gate="1" pin="GND"/>
 <pinref part="RN2" gate="A" pin="1"/>
-<wire x1="104.14" y1="728.98" x2="106.68" y2="728.98" width="0.1524" layer="91"/>
+<wire x1="104.14" y1="728.98" x2="109.22" y2="728.98" width="0.1524" layer="91"/>
 </segment>
 <segment>
@@
 <label x="477.52" y="480.06" size="1.778" layer="95"/>
 </segment>
-<segment>
-<pinref part="U$125" gate="G$1" pin="A-B"/>
-<wire x1="327.66" y1="157.48" x2="312.42" y2="157.48" width="0.1524" layer="91"/>
-<label x="312.42" y="157.48" size="1.778" layer="95"/>
-</segment>
 </net>
 <net name="N6_A4_SDA" class="0">
@@
 <label x="477.52" y="99.06" size="1.778" layer="95"/>
 </segment>
+<segment>
+<pinref part="U$125" gate="G$1" pin="A-B"/>
+<wire x1="327.66" y1="157.48" x2="312.42" y2="157.48" width="0.1524" layer="91"/>
+<label x="312.42" y="157.48" size="1.778" layer="95"/>
+</segment>
 </net>

Commit message: Routing
Other:
- note added: "MCP23017 can supply 25mA per output. Directly control node VCCs?"
- note removed: "Add FETs or something to switch node VCCs?"
- note removed: "Control UART switch EN from supervisor"
- note removed: "MCP23017 can only supply 25mA per output."
- note removed: "May not be suitable for direct control of node VCCs."
- note removed: "Replace 2 x MCP23017 with 1 x ATmega328?"
Changed lines of the file:
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@@
 <text x="53.34" y="622.3" size="1.778" layer="94">I2C Isolation</text>
 <text x="53.34" y="660.4" size="1.778" layer="94">Status Display</text>
-<text x="99.06" y="843.28" size="1.778" layer="94">MCP23017 can only supply 25mA per output.</text>
-<text x="99.06" y="840.74" size="1.778" layer="94">May not be suitable for direct control of node VCCs.</text>
-<text x="99.06" y="833.12" size="1.778" layer="94">Replace 2 x MCP23017 with 1 x ATmega328?</text>
+<text x="99.06" y="843.28" size="1.778" layer="94">MCP23017 can supply 25mA per output. Directly control node VCCs?</text>
 <wire x1="73.66" y1="942.34" x2="73.66" y2="894.08" width="0.1524" layer="97" style="longdash"/>
 <wire x1="73.66" y1="894.08" x2="73.66" y2="782.32" width="0.1524" layer="97" style="longdash"/>
 <wire x1="73.66" y1="782.32" x2="73.66" y2="767.08" width="0.1524" layer="97" style="longdash"/>
 <text x="83.82" y="939.038" size="1.778" layer="94">I2C Bias: Management Bus</text>
-<text x="99.06" y="838.2" size="1.778" layer="94">Add FETs or something to switch node VCCs?</text>
 <text x="99.06" y="828.04" size="1.778" layer="94">What bus pins to use for UART, I2C, and MGMNT_I2C?</text>
 <text x="99.06" y="825.5" size="1.778" layer="94">Add bias for MGMNT_I2C</text>
@@
 <text x="7.62" y="581.66" size="3.81" layer="94">Node 1</text>
 <text x="7.62" y="586.74" size="3.81" layer="94">Processor</text>
-<text x="99.06" y="820.42" size="1.778" layer="94">Control UART switch EN from supervisor</text>
 <text x="99.06" y="800.1" size="1.778" layer="94">Pass through RESET for each node? Easy, but better perhaps
 to expose one of the Supervisor node I/O lines as a "virtual"

Commit message: Routing
Parts:
- P5: device freetronics-jon:ICSPSMT -> freetronics-jon:ICSPPTH
Changed lines of the file:
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@@
 <part name="R26" library="freetronics-master-v1.1" deviceset="RESISTOR" device="0603" value="22K 0603"/>
 <part name="U$51" library="SparkFun" deviceset="5V" device=""/>
-<part name="P5" library="freetronics-jon" deviceset="ICSP" device="SMT" value="N1_ICSP"/>
+<part name="P5" library="freetronics-jon" deviceset="ICSP" device="PTH" value="N1_ICSP"/>
 <part name="GND29" library="SparkFun" deviceset="GND" device=""/>
 <part name="U$52" library="SparkFun" deviceset="5V" device=""/>
