File: ArduSatPayloadModule.brd (EAGLE design)
At the start: 95.5 x 90.3 mm, 304 parts, among them IC1 ATMEGA328P QFN32, IC10 ATMEGA328P QFN32, IC11 ATMEGA328P QFN32, IC12 ATMEGA328P QFN32, IC13 ATMEGA328P QFN32, IC14 ATMEGA328P QFN32, IC15 ATMEGA328P QFN32, IC16 ATMEGA328P QFN32, IC17 DS3232, IC2 ATMEGA328P QFN32, IC20 ATMEGA2561-16MU, IC3 ATMEGA328P QFN32, IC4 ATMEGA328P QFN32, IC5 ATMEGA328P QFN32, IC6 ATMEGA328P QFN32, IC7 ATMEGA328P QFN32, IC8 ATMEGA328P QFN32, IC9 ATMEGA328P QFN32, P14 microSD, P5 S_ICSP, Q1 RJU003N03 N-MOSFET, Q10 RJU003N03 N-MOSFET, Q11 RJU003N03 N-MOSFET, Q12 RJU003N03 N-MOSFET, Q13 RJU003N03 N-MOSFET, Q14 RJU003N03 N-MOSFET, Q15 RJU003N03 N-MOSFET, Q16 RJU003N03 N-MOSFET, Q17 RJU003N03 N-MOSFET, Q18 RJU003N03 N-MOSFET, Q19 RJU003N03 N-MOSFET, Q2 RJU003N03 N-MOSFET, Q20 RJU003N03 N-MOSFET, Q21 RJU003N03 N-MOSFET, Q22 RJU003N03 N-MOSFET, Q23 RJU003N03 N-MOSFET, Q24 RJU003N03 N-MOSFET, Q25 RJU003N03 N-MOSFET, Q26 RJU003N03 N-MOSFET, Q27 RJU003N03 N-MOSFET, Q28 RJU003N03 N-MOSFET, Q29 RJU003N03 N-MOSFET, Q3 RJU003N03 N-MOSFET, Q30 RJU003N03 N-MOSFET, Q31 RJU003N03 N-MOSFET, Q32 RJU003N03 N-MOSFET, Q33 RJU003N03 N-MOSFET, Q34 RJU003N03 N-MOSFET, Q35 RJU003N03 N-MOSFET, Q36 RJU003N03 N-MOSFET, Q37 RJU003N03 N-MOSFET, Q38 RJU003N03 N-MOSFET, Q39 RJU003N03 N-MOSFET, Q4 RJU003N03 N-MOSFET, Q40 RJU003N03 N-MOSFET, Q41 RJU003N03 N-MOSFET, Q42 RJU003N03 N-MOSFET, Q5 RJU003N03 N-MOSFET, Q6 RJU003N03 N-MOSFET, Q7 RJU003N03 N-MOSFET, Q8 RJU003N03 N-MOSFET, Q9 RJU003N03 N-MOSFET, SW1 ADG801SOT23-6, SW10 ADG801SOT23-6, SW11 ADG801SOT23-6, SW12 ADG801SOT23-6, SW13 ADG801SOT23-6, SW14 ADG801SOT23-6, SW15 ADG801SOT23-6, SW16 ADG801SOT23-6, SW2 ADG801SOT23-6, SW3 ADG801SOT23-6, SW4 ADG801SOT23-6, SW5 ADG801SOT23-6, SW6 ADG801SOT23-6, SW7 ADG801SOT23-6, SW8 ADG801SOT23-6, SW9 ADG801SOT23-6, X1 geiger, X2 gps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

Commit message: Placement and routing
Parts:
- removed C58: 100nF, freetronics-jon:0402C
- removed IC17: DS3232, freetronics-master-v1:SO20L
- removed Q37, Q38: RJU003N03 N-MOSFET, freetronics-jon:SOT32-3
- removed R81, R82: 4K7 0402, freetronics-jon:0402
- removed U$21, U$22: FIDUCIAL1X2.5, freetronics:FIDUCIAL-1X2.5
- added C59, C60: 10uF 10V A TANT, freetronics:EIA3216
- added C61, C62: 100nF 0402, freetronics-jon:0402C
- added FID1, FID2, FID3, FID4: FIDUCIAL1X2.5, freetronics:FIDUCIAL-1X2.5
- added IC18, IC19: TMP102, freetronics-jon:SOT563
- added R83, R84, R85, R86: 10K 0402, freetronics-jon:0402
- added S1: RESET, freetronics-master-v1:TACTILE_SWITCH_SMD_2PIN_TINY
- added U$29, U$30, U$31, U$32: MOSFET-NSOT-323, freetronics-jon:SOT32-3
- added U$33: (no value), OSHW:OSHW_10X200_NOTEXT
- C39: device freetronics:0603 -> freetronics-jon:0402C
- IC20: device atmel-2005:MLF64 -> freetronics-jon:MLF64
- R4, R5: value 100K 0402 -> 10K 0402
- moved U$26 124.8 mm to (46.2, 28.4), flipped to the bottom, turned to 270 degrees
- moved R80 108.0 mm to (54.1, 6.86), flipped to the bottom, turned to 90 degrees
- moved Q42 107.1 mm to (52.1, 6.86), flipped to the bottom, turned to 270 degrees
- moved Q41 106.8 mm to (52.6, 9.91), flipped to the bottom, turned to 270 degrees
- moved Q35 105.3 mm to (43.7, 45.5), flipped to the bottom, turned to 270 degrees
- moved R21 104.3 mm to (46.0, 48.5), flipped to the bottom, turned to 90 degrees
- moved Q36 103.3 mm to (43.7, 48.5), flipped to the bottom, turned to 270 degrees
- moved C2 103.2 mm to (4.32, 62.5)
- moved C3 103.2 mm to (4.83, 57.1)
- moved H3 103.2 mm to (10.9, 58.4)
- moved IC1 103.2 mm to (10.9, 63.8)
- moved LED1 103.2 mm to (4.32, 64.8)
- moved Q1 103.2 mm to (16.8, 65.0)
- moved Q2 103.2 mm to (16.8, 67.6)
- moved R2 103.2 mm to (7.11, 61.2)
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Connections:
- removed net 3V3D: C39.1, P14.4
- removed net 3V3_GPS: U$26.1, U$26.12, X2.2
- removed net 5V_GPS: X2.1
- removed net N$10000: IC17.17, Q37.2, R81.1
- removed net N$9998: IC17.18, IC17.20, Q38.2, R82.1
- removed net S_D2: IC20.6
- removed net S_D3: IC20.7
- removed net S_D5: IC20.5
- new net N$10001: IC18.6, R84.1, U$30.2
- new net N$10002: IC19.6, R86.1, U$32.2
- new net N$10003: IC19.1, R85.1, U$31.2
- new net N$9999: IC18.1, R83.1, U$29.2
- net 3.3V: now also C39.1, C59.A, C61.1, C62.1, IC18.5, IC19.4, IC19.5, P14.4, R83.2, R84.2, R85.2, R86.2, U$26.1, U$26.12, U$29.1, U$30.1, U$31.1, U$32.1, X1.5, X2.2, X4.6, X6.4
- net 5V: now also C60.A, JP4.2, X2.1; no longer C58.1, IC17.4, Q37.1, Q38.1, R81.2, R82.2
- net GND: now also C59.C, C60.C, C61.2, C62.2, IC18.2, IC18.4, IC19.2, IC20.TGND1, IC20.TGND2, IC20.TGND3, IC20.TGND4, S1.1; no longer C58.2, IC17.1, IC17.10, IC17.11, IC17.12, IC17.13, IC17.14, IC17.15, IC17.16, IC17.19, IC17.2, IC17.7, IC17.8, IC17.9
- net N$23: now also RN14.2; no longer RN14.4
- net N$321: now also RN13.6, RN14.4; no longer RN13.7, RN14.2
- net N$90: now also RN13.7; no longer RN13.6
- net PWR_GEIGER: now also IC20.5
- net PWR_SPEC: now also IC20.6
- net RST_SPEC: now also IC20.7
- net SCL: now also U$29.3, U$31.3; no longer Q38.3
- net SDA: now also U$30.3, U$32.3; no longer Q37.3
- net S_D10: now also RN14.7; no longer RN14.5
- net S_D52_SCK: now also RN14.5; no longer RN14.7
- net S_RESET: now also S1.2
- net VCC_SYS: no longer JP4.2, X1.5, X4.6, X6.4
Routing:
- net 5V: track 83.1 -> 600.1 mm, vias 0 -> 18
- net SDA: track 29.9 -> 424.1 mm, vias 16 -> 19
- net SCL: track 29.9 -> 393.3 mm, vias 16 -> 19
- net 3.3V: track 0.00 -> 283.8 mm, vias 0 -> 3
- net S_A1: track 0.00 -> 80.2 mm, vias 0 -> 2
- net S_A4: track 0.00 -> 66.1 mm, vias 0 -> 3
- net S_A3: track 0.00 -> 63.8 mm, vias 0 -> 3
- net PWR_SPEC: track 0.00 -> 61.1 mm, vias 0 -> 1
- net S_A0: track 0.00 -> 59.9 mm, vias 0 -> 2
- net S_A5: track 0.00 -> 59.5 mm, vias 0 -> 3
- net N13_D1_TX: track 40.9 -> 97.9 mm, vias 1 -> 2
- net RST_SPEC: track 0.00 -> 55.2 mm, vias 0 -> 1
- net N16_D0_RX: track 22.2 -> 77.2 mm, vias 1 -> 2
- net N16_D1_TX: track 40.9 -> 94.2 mm, vias 1 -> 2
- net S_A6: track 0.00 -> 50.3 mm, vias 0 -> 3
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Other:
- board text added: "/Users/jon/Dropbox/Freetronics/ConsultingProjects/ArduSat/nanosatisfi 2-2 BW.bmp"
- board text added: "ArduSat Payload Processor Module"
- board text added: "Main I2C bus"
- board text added: "PWR"
- board text added: "RESET"
- board text added: "by Jon Oxer"
- board text added: "pullups (opt)"
- board text added: "www.ardusat.org"
- board text removed: "Freetronics ArduSat Payload Processor Module"
- board text removed: "RTC"
