File: ArduSatPayloadModule.sch (EAGLE design)
At the start: 304 parts, among them IC1 ATMEGA328P QFN32, IC10 ATMEGA328P QFN32, IC11 ATMEGA328P QFN32, IC12 ATMEGA328P QFN32, IC13 ATMEGA328P QFN32, IC14 ATMEGA328P QFN32, IC15 ATMEGA328P QFN32, IC16 ATMEGA328P QFN32, IC17 DS3232, IC2 ATMEGA328P QFN32, IC20 ATMEGA2561-16MU, IC3 ATMEGA328P QFN32, IC4 ATMEGA328P QFN32, IC5 ATMEGA328P QFN32, IC6 ATMEGA328P QFN32, IC7 ATMEGA328P QFN32, IC8 ATMEGA328P QFN32, IC9 ATMEGA328P QFN32, P14 microSD, P5 S_ICSP, Q1 RJU003N03 N-MOSFET, Q10 RJU003N03 N-MOSFET, Q11 RJU003N03 N-MOSFET, Q12 RJU003N03 N-MOSFET, Q13 RJU003N03 N-MOSFET, Q14 RJU003N03 N-MOSFET, Q15 RJU003N03 N-MOSFET, Q16 RJU003N03 N-MOSFET, Q17 RJU003N03 N-MOSFET, Q18 RJU003N03 N-MOSFET, Q19 RJU003N03 N-MOSFET, Q2 RJU003N03 N-MOSFET, Q20 RJU003N03 N-MOSFET, Q21 RJU003N03 N-MOSFET, Q22 RJU003N03 N-MOSFET, Q23 RJU003N03 N-MOSFET, Q24 RJU003N03 N-MOSFET, Q25 RJU003N03 N-MOSFET, Q26 RJU003N03 N-MOSFET, Q27 RJU003N03 N-MOSFET, Q28 RJU003N03 N-MOSFET, Q29 RJU003N03 N-MOSFET, Q3 RJU003N03 N-MOSFET, Q30 RJU003N03 N-MOSFET, Q31 RJU003N03 N-MOSFET, Q32 RJU003N03 N-MOSFET, Q33 RJU003N03 N-MOSFET, Q34 RJU003N03 N-MOSFET, Q35 RJU003N03 N-MOSFET, Q36 RJU003N03 N-MOSFET, Q37 RJU003N03 N-MOSFET, Q38 RJU003N03 N-MOSFET, Q39 RJU003N03 N-MOSFET, Q4 RJU003N03 N-MOSFET, Q40 RJU003N03 N-MOSFET, Q41 RJU003N03 N-MOSFET, Q42 RJU003N03 N-MOSFET, Q5 RJU003N03 N-MOSFET, Q6 RJU003N03 N-MOSFET, Q7 RJU003N03 N-MOSFET, Q8 RJU003N03 N-MOSFET, Q9 RJU003N03 N-MOSFET, SW1 ADG801SOT23-6, SW10 ADG801SOT23-6, SW11 ADG801SOT23-6, SW12 ADG801SOT23-6, SW13 ADG801SOT23-6, SW14 ADG801SOT23-6, SW15 ADG801SOT23-6, SW16 ADG801SOT23-6, SW2 ADG801SOT23-6, SW3 ADG801SOT23-6, SW4 ADG801SOT23-6, SW5 ADG801SOT23-6, SW6 ADG801SOT23-6, SW7 ADG801SOT23-6, SW8 ADG801SOT23-6, SW9 ADG801SOT23-6, X1 geiger, X2 gps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

Commit message: Placement and routing
Parts:
- removed C58: 100nF, freetronics-jon:C-EU0402C
- removed IC17: DS3232, freetronics-master-v1:DS3232
- removed Q37, Q38: RJU003N03 N-MOSFET, freetronics-jon:MOSFET-NSOT-323
- removed R81, R82: 4K7 0402, freetronics-jon:RESISTOR0402
- removed U$21, U$22: FIDUCIAL1X2.5, freetronics:FIDUCIAL1X2.5
- added C59, C60: 10uF 10V A TANT, freetronics:CAP_POL1206
- added C61, C62: 100nF 0402, freetronics-jon:C-EU0402C
- added FID1, FID2, FID3, FID4: FIDUCIAL1X2.5, freetronics:FIDUCIAL1X2.5
- added IC18, IC19: TMP102, freetronics-jon:TMP102
- added R83, R84, R85, R86: 10K 0402, freetronics-jon:RESISTOR0402
- added S1: RESET, freetronics-master-v1:TAC_SWITCH_2PIN
- added U$29, U$30, U$31, U$32: MOSFET-NSOT-323, freetronics-jon:MOSFET-NSOT-323
- C39: device freetronics:CAP0603 -> freetronics-jon:C-EU0402C
- IC20: device atmel-2005:ATMEGA2561-16MU -> freetronics-jon:ATMEGA2561-16MU
- R4, R5: value 100K 0402 -> 10K 0402
Connections:
- removed net 3V3D: C39.1, P14.VCC
- removed net 3V3_GPS: U$26.OE, U$26.VCCA, X2-2.S
- removed net 5V_GPS: X2-1.S
- removed net N$10000: IC17.SDA, Q37.S, R81.1
- removed net N$9998: IC17.SCL@18, IC17.SCL@20, Q38.S, R82.1
- removed net S_D2: IC20.(OC3B/INT4)PE4
- removed net S_D3: IC20.(OC3C/INT5)PE5
- removed net S_D5: IC20.(OC3A/AIN1)PE3
- new net N$10001: IC18.SDA, R84.1, U$30.S
- new net N$10002: IC19.SDA, R86.1, U$32.S
- new net N$10003: IC19.SCL, R85.1, U$31.S
- new net N$9999: IC18.SCL, R83.1, U$29.S
- net 3.3V: now also C39.1, C59.+, C61.1, C62.1, IC18.V+, IC19.ADD0, IC19.V+, P14.VCC, R83.2, R84.2, R85.2, R86.2, U$26.OE, U$26.VCCA, U$29.G, U$30.G, U$31.G, U$32.G, X1-5.S, X2-2.S, X4-6.S, X6-4.S
- net 5V: now also C60.+, JP4.2, X2-1.S; no longer C58.1, IC17.VCC, Q37.G, Q38.G, R81.2, R82.2
- net GND: now also C59.-, C60.-, C61.2, C62.2, IC18.ADD0, IC18.GND, IC19.GND, IC20.TGND1, IC20.TGND2, IC20.TGND3, IC20.TGND4, S1.P; no longer C58.2, IC17.GND, IC17.NC@1, IC17.NC@10, IC17.NC@11, IC17.NC@12, IC17.NC@13, IC17.NC@14, IC17.NC@19, IC17.NC@2, IC17.NC@7, IC17.NC@8, IC17.NC@9, IC17.VBAT
- net N$23: now also RN14B.1; no longer RN14D.1
- net N$321: now also RN13C.2, RN14D.1; no longer RN13B.2, RN14B.1
- net N$90: now also RN13B.2; no longer RN13C.2
- net PWR_GEIGER: now also IC20.(OC3A/AIN1)PE3
- net PWR_SPEC: now also IC20.(OC3B/INT4)PE4
- net RST_SPEC: now also IC20.(OC3C/INT5)PE5
- net SCL: now also U$29.D, U$31.D; no longer Q38.D
- net SDA: now also U$30.D, U$32.D; no longer Q37.D
- net S_D10: now also RN14B.2; no longer RN14D.2
- net S_D52_SCK: now also RN14D.2; no longer RN14B.2
- net S_RESET: now also S1.S
- net VCC_SYS: no longer JP4.2, X1-5.S, X4-6.S, X6-4.S
Other:
- note added: "Bottom Temperature Sensor"
- note added: "Debug was connected to VCC_SYS, I switched it to 5V. Is that OK?"
- note added: "GPS is susceptible to supply ripple. Extra decoupling or a filter to remove switching supply noise?"
- note added: "I2C Addr: 72 (0x48)"
- note added: "I2C Addr: 73 (0x49)"
- note added: "Note: GPS is connected via serial level shifters to processor node 11"
- note added: "S_D2"
- note added: "S_D3"
- note added: "S_D5"
- note added: "Top Temperature Sensor"
- note added: "V1.0 (2013-01-07)"
- note removed: "I2C address = 0x68. VBAT connected to GND because no battery used. Accuracy +/-2ppm from 0 to 40 deg. C. Onboard temperature sensor +/-3 deg. C."
- note removed: "V1.0 (2013-01-02)"
- moved on the sheet: C39, JP4, MNT1, MNT2, MNT3, MNT4, P14, P5, R26, RN13A, RN13B, RN13C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
