File: ArduSatPayloadProcessorModule.sch (EAGLE design)
At the start: 315 parts, among them IC1 ATMEGA328P QFN32, IC10 ATMEGA328P QFN32, IC11 ATMEGA328P QFN32, IC12 ATMEGA328P QFN32, IC13 ATMEGA328P QFN32, IC14 ATMEGA328P QFN32, IC15 ATMEGA328P QFN32, IC16 ATMEGA328P QFN32, IC18 TMP102, IC19 TMP102, IC2 ATMEGA328P QFN32, IC20 ATMEGA2561-16MU, IC3 ATMEGA328P QFN32, IC4 ATMEGA328P QFN32, IC5 ATMEGA328P QFN32, IC6 ATMEGA328P QFN32, IC7 ATMEGA328P QFN32, IC8 ATMEGA328P QFN32, IC9 ATMEGA328P QFN32, P14 microSD, P5 S_ICSP, Q1 RJU003N03 N-MOSFET, Q10 RJU003N03 N-MOSFET, Q11 RJU003N03 N-MOSFET, Q12 RJU003N03 N-MOSFET, Q13 RJU003N03 N-MOSFET, Q14 RJU003N03 N-MOSFET, Q15 RJU003N03 N-MOSFET, Q16 RJU003N03 N-MOSFET, Q17 RJU003N03 N-MOSFET, Q18 RJU003N03 N-MOSFET, Q19 RJU003N03 N-MOSFET, Q2 RJU003N03 N-MOSFET, Q20 RJU003N03 N-MOSFET, Q21 RJU003N03 N-MOSFET, Q22 RJU003N03 N-MOSFET, Q23 RJU003N03 N-MOSFET, Q24 RJU003N03 N-MOSFET, Q25 RJU003N03 N-MOSFET, Q26 RJU003N03 N-MOSFET, Q27 RJU003N03 N-MOSFET, Q28 RJU003N03 N-MOSFET, Q29 RJU003N03 N-MOSFET, Q3 RJU003N03 N-MOSFET, Q30 RJU003N03 N-MOSFET, Q31 RJU003N03 N-MOSFET, Q32 RJU003N03 N-MOSFET, Q33 RJU003N03 N-MOSFET, Q34 RJU003N03 N-MOSFET, Q35 RJU003N03 N-MOSFET, Q36 RJU003N03 N-MOSFET, Q39 RJU003N03 N-MOSFET, Q4 RJU003N03 N-MOSFET, Q40 RJU003N03 N-MOSFET, Q41 RJU003N03 N-MOSFET, Q42 RJU003N03 N-MOSFET, Q5 RJU003N03 N-MOSFET, Q6 RJU003N03 N-MOSFET, Q7 RJU003N03 N-MOSFET, Q8 RJU003N03 N-MOSFET, Q9 RJU003N03 N-MOSFET, SW1 ADG801SOT23-6, SW10 ADG801SOT23-6, SW11 ADG801SOT23-6, SW12 ADG801SOT23-6, SW13 ADG801SOT23-6, SW14 ADG801SOT23-6, SW15 ADG801SOT23-6, SW16 ADG801SOT23-6, SW2 ADG801SOT23-6, SW3 ADG801SOT23-6, SW4 ADG801SOT23-6, SW5 ADG801SOT23-6, SW6 ADG801SOT23-6, SW7 ADG801SOT23-6, SW8 ADG801SOT23-6, SW9 ADG801SOT23-6, X1 geiger, X2 gps, X4 spectruino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

Commit message: ERC and DRC for production
Parts:
- removed X6: 53398-04, con-molex:53398-04
- added X3: Spectruino, con-molex:53398-07
- C40, C51: device freetronics-master-v1.1:CAP0603 -> freetronics-jon:C-EU0402C
- IC21, IC22: value MAX4372 -> MAX4372F
- JP1: value (none) -> DEBUG
- LED17: value RGBLEDSMT -> BLUE 0603; device freetronics-jon:RGBLEDSMT -> freetronics:LED0603
- LED4: value PWR/BLUE -> RGBLEDSMT; device freetronics:LED0603 -> freetronics-jon:RGBLEDSMT
- Q43, Q44, Q45, Q46: value MOSFET-NSOT-323 -> RJU003N03 N-MOSFET
- R59, R75: value 0.15R 2010 -> 0.1R 2010
- RN13: device freetronics-master-v1:4R-NCAY16 -> resistor-dil:4R-NCAY16
- RN14: value 1K -> 2K2; device freetronics-master-v1:4R-NCAY16 -> resistor-dil:4R-NCAY16
- RN17: device resistor-dil:4R-NCAY16 -> freetronics-master-v1:4R-NCAY16
- RN18: value 2K2 -> 1K; device resistor-dil:4R-NCAY16 -> freetronics-master-v1:4R-NCAY16
- SW1, SW10, SW11, SW12, SW13, SW14, SW15, SW16, SW2, SW3, SW4, SW5, SW6, SW7, SW8, SW9: value ADG801SOT23-6 -> ADG801 SOT23-6
- X1: value geiger -> Geiger
- X4: value spectruino -> Bottom Plate; device con-molex:53398-07 -> con-molex:53398-04
- XTL17: value CRYSTAL-GND3X2 -> SMD3225-16MHZ 3.2 x 2.5mm crystal
- renumbered JP4 to JP1, P14 to P1, P5 to H19, S1 to SW17, U$156 to IC21, U$26 to IC17, U$29 to Q43, U$30 to Q44, U$31 to Q45, U$32 to Q46, U$34 to IC22, U$53 to XTL17, U$59 to IC24, U$60 to IC23
Connections:
- removed net RX: IC24.Z
- removed net S_D38: IC20.(T0)PD7
- removed net TX: IC23.Z
- net 3.3V: now also X3-6.S, X4-4.S; no longer X4-6.S, X6-4.S
- net 5V: now also LED17.A, X3-1.S; no longer LED4.A, X4-1.S
- net BOTTOM_SCL: now also X4-1.S; no longer X6-1.S
- net BOTTOM_SDA: now also X4-2.S; no longer X6-2.S
- net D0_RX: now also IC24.Z
- net D1_TX: now also IC23.Z
- net GND: now also RN14A.1, RN17B.1, RN17C.1, X3-7.S, X4-3.S; no longer RN13B.1, RN13C.1, RN18A.1, X4-7.S, X6-3.S
- net N$14: now also LED17.C; no longer LED4.C
- net N$23: now also RN17A.2, RN18B.1; no longer RN13A.2, RN14B.1
- net N$2356: now also LED4.C-R; no longer LED5.C-R
- net N$2357: now also LED4.C-B; no longer LED5.C-B
- net N$2358: now also LED4.C-G; no longer LED5.C-G
- net N$2944: now also LED5.C-R; no longer LED6.C-R
- net N$2945: now also LED5.C-B; no longer LED6.C-B
- net N$2946: now also LED5.C-G; no longer LED6.C-G
- net N$321: now also RN17C.2, RN18D.1; no longer RN13C.2, RN14D.1
- net N$3532: now also LED6.C-R; no longer LED7.C-R
- net N$3533: now also LED6.C-B; no longer LED7.C-B
- net N$3534: now also LED6.C-G; no longer LED7.C-G
- net N$4120: now also LED7.C-R; no longer LED8.C-R
- net N$4121: now also LED7.C-B; no longer LED8.C-B
- net N$4122: now also LED7.C-G; no longer LED8.C-G
- net N$4708: now also LED8.C-R; no longer LED9.C-R
- net N$4709: now also LED8.C-B; no longer LED9.C-B
- net N$4710: now also LED8.C-G; no longer LED9.C-G
- net N$5296: now also LED9.C-R; no longer LED10.C-R
- net N$5297: now also LED9.C-B; no longer LED10.C-B
- net N$5298: now also LED9.C-G; no longer LED10.C-G
- net N$5884: now also LED10.C-R; no longer LED11.C-R
- net N$5885: now also LED10.C-B; no longer LED11.C-B
- net N$5886: now also LED10.C-G; no longer LED11.C-G
- net N$6472: now also LED11.C-R; no longer LED12.C-R
- net N$6473: now also LED11.C-B; no longer LED12.C-B
- net N$6474: now also LED11.C-G; no longer LED12.C-G
- net N$7060: now also LED12.C-R; no longer LED13.C-R
- net N$7061: now also LED12.C-B; no longer LED13.C-B
- net N$7062: now also LED12.C-G; no longer LED13.C-G
- net N$7648: now also LED13.C-R, RN13B.2; no longer LED14.C-R, RN15B.2
- net N$7649: now also LED13.C-B, RN13A.2; no longer LED14.C-B, RN15A.2
- net N$7650: now also LED13.C-G, RN13D.2; no longer LED14.C-G, RN15D.2
- net N$8236: now also LED14.C-R, RN14B.2; no longer LED15.C-R, RN16B.2
- net N$8237: now also LED14.C-B, RN14A.2; no longer LED15.C-B, RN16A.2
- net N$8238: now also LED14.C-G, RN14D.2; no longer LED15.C-G, RN16D.2
- net N$8824: now also LED15.C-R, RN15B.2; no longer LED16.C-R, RN17B.2
- net N$8825: now also LED15.C-B, RN15A.2; no longer LED16.C-B, RN17A.2
- net N$8826: now also LED15.C-G, RN15D.2; no longer LED16.C-G, RN17D.2
- net N$90: now also RN17B.2, RN18C.1; no longer RN13B.2, RN14C.1
- net N$9412: now also LED16.C-R, RN16B.2; no longer LED17.C-R, RN18B.2
- net N$9413: now also LED16.C-B, RN16A.2; no longer LED17.C-B, RN18A.2
- net N$9414: now also LED16.C-G, RN16D.2; no longer LED17.C-G, RN18D.2
- net N10_5V: now also LED10.A-G, LED10.A-R; no longer LED11.A-G, LED11.A-R
- net N10_D13_SCK: now also LED10.A-B; no longer LED11.A-B
- net N11_5V: now also LED11.A-G, LED11.A-R; no longer LED12.A-G, LED12.A-R
- net N11_D13_SCK: now also LED11.A-B; no longer LED12.A-B
- net N12_5V: now also LED12.A-G, LED12.A-R; no longer LED13.A-G, LED13.A-R
- net N12_D13_SCK: now also LED12.A-B; no longer LED13.A-B
- net N13_5V: now also LED13.A-G, LED13.A-R; no longer LED14.A-G, LED14.A-R
- net N13_D0_RX: now also RN13D.1; no longer RN15D.1
- net N13_D13_SCK: now also LED13.A-B; no longer LED14.A-B
- net N13_D1_TX: now also RN13B.1; no longer RN15B.1
- net N14_5V: now also LED14.A-G, LED14.A-R; no longer LED15.A-G, LED15.A-R
- net N14_D0_RX: now also RN14D.1; no longer RN16D.1
- net N14_D13_SCK: now also LED14.A-B; no longer LED15.A-B
- net N14_D1_TX: now also RN14B.1; no longer RN16B.1
- net N15_5V: now also LED15.A-G, LED15.A-R; no longer LED16.A-G, LED16.A-R
- net N15_D0_RX: now also RN15D.1; no longer RN17D.1
- net N15_D13_SCK: now also LED15.A-B; no longer LED16.A-B
- net N15_D1_TX: now also RN15B.1; no longer RN17B.1
- net N16_5V: now also LED16.A-G, LED16.A-R; no longer LED17.A-G, LED17.A-R
- net N16_D0_RX: now also RN16D.1; no longer RN18D.1
- net N16_D13_SCK: now also LED16.A-B; no longer LED17.A-B
- net N16_D1_TX: now also RN16B.1; no longer RN18B.1
- net N4_5V: now also LED4.A-G, LED4.A-R; no longer LED5.A-G, LED5.A-R
- net N4_D13_SCK: now also LED4.A-B; no longer LED5.A-B
- net N5_5V: now also LED5.A-G, LED5.A-R; no longer LED6.A-G, LED6.A-R
- net N5_D13_SCK: now also LED5.A-B; no longer LED6.A-B
- net N6_5V: now also LED6.A-G, LED6.A-R; no longer LED7.A-G, LED7.A-R
- net N6_D13_SCK: now also LED6.A-B; no longer LED7.A-B
- net N7_5V: now also LED7.A-G, LED7.A-R; no longer LED8.A-G, LED8.A-R
- net N7_D13_SCK: now also LED7.A-B; no longer LED8.A-B
- net N8_5V: now also LED8.A-G, LED8.A-R; no longer LED9.A-G, LED9.A-R
- net N8_D13_SCK: now also LED8.A-B; no longer LED9.A-B
- net N9_5V: now also LED9.A-G, LED9.A-R; no longer LED10.A-G, LED10.A-R
- net N9_D13_SCK: now also LED9.A-B; no longer LED10.A-B
- net PWR_SPEC: now also X3-2.S; no longer X4-2.S
- net RST_GPS: now also IC20.(T0)PD7
- net RST_SPEC: now also X3-3.S; no longer X4-3.S
- net SPEC_SCL: now also X3-5.S; no longer X4-5.S
- net SPEC_SDA: now also X3-4.S; no longer X4-4.S
- net S_D10: now also RN18B.2; no longer RN14B.2
- net S_D51_MOSI: now also RN18C.2; no longer RN14C.2
- net S_D52_SCK: now also RN18D.2; no longer RN14D.2
Other:
- note added: "3.3V Current Sensor (0-1A)"
- note added: "5V Current Sensor (0-1A)"
- note added: "Debug console"
- note added: "S_D38"
- note removed: "3.3V Current Sensor"
- note removed: "5V Current Sensor"
- note removed: "Add power links for GPS, Geiger, Spectruino, Bottom Plate"
- note removed: "Add status LEDs to the MUX address and enable lines?"
- note removed: "Pass through RESET for each node? Easy, but better perhaps to expose one of the Supervisor node I/O lines as a "virtual" reset line, which in turn toggles power to that node. That way the interface to this board externally just looks like TX, RX, and RESET, like any other Arduino. It would just need the node selected first."
- note removed: "What bus pins to use for UART, I2C, and MGMNT_I2C?"
- moved on the sheet: C40, C51, X4-1, X4-2, X4-3, X4-4

Commit message: Fix footprint for RGB LED
Parts:
- LED1, LED10, LED11, LED12, LED13, LED14, LED15, LED16, LED2, LED3, LED4, LED5, LED6, LED7, LED8, LED9: value RGBLEDSMT -> FREETRONICS-MASTER-V1_RGBLEDSMT; device freetronics-jon:RGBLEDSMT -> freetronics-master-v1:FREETRONICS-MASTER-V1_RGBLEDSMT
Changed lines of the file:
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@@
 <part name="R2" library="freetronics-jon" deviceset="RESISTOR" device="0402" value="1M 0402"/>
 <part name="XTL1" library="freetronics-jon" deviceset="CRYSTAL-GND" device="3X2" value="SMD3225-16MHZ 3.2 x 2.5mm crystal"/>
-<part name="LED1" library="freetronics-jon" deviceset="RGBLED" device="SMT"/>
+<part name="LED1" library="freetronics-master-v1" deviceset="FREETRONICS-MASTER-V1_RGBLED" device="SMT"/>
 <part name="RN1" library="resistor-dil" deviceset="4R-N" device="CAY16" value="2K2"/>
 <part name="GND87" library="SparkFun" deviceset="GND" device=""/>
@@
 <part name="R8" library="freetronics-jon" deviceset="RESISTOR" device="0402" value="1M 0402"/>
 <part name="XTL2" library="freetronics-jon" deviceset="CRYSTAL-GND" device="3X2" value="SMD3225-16MHZ 3.2 x 2.5mm crystal"/>
-<part name="LED2" library="freetronics-jon" deviceset="RGBLED" device="SMT"/>
+<part name="LED2" library="freetronics-master-v1" deviceset="FREETRONICS-MASTER-V1_RGBLED" device="SMT"/>
 <part name="RN2" library="resistor-dil" deviceset="4R-N" device="CAY16" value="2K2"/>
 <part name="GND6" library="SparkFun" deviceset="GND" device=""/>
@@
 <part name="R13" library="freetronics-jon" deviceset="RESISTOR" device="0402" value="1M 0402"/>
 <part name="XTL3" library="freetronics-jon" deviceset="CRYSTAL-GND" device="3X2" value="SMD3225-16MHZ 3.2 x 2.5mm crystal"/>
-<part name="LED3" library="freetronics-jon" deviceset="RGBLED" device="SMT"/>
+<part name="LED3" library="freetronics-master-v1" deviceset="FREETRONICS-MASTER-V1_RGBLED" device="SMT"/>
 <part name="RN3" library="resistor-dil" deviceset="4R-N" device="CAY16" value="2K2"/>
 <part name="GND11" library="SparkFun" deviceset="GND" device=""/>
@@
 <part name="R17" library="freetronics-jon" deviceset="RESISTOR" device="0402" value="1M 0402"/>
 <part name="XTL4" library="freetronics-jon" deviceset="CRYSTAL-GND" device="3X2" value="SMD3225-16MHZ 3.2 x 2.5mm crystal"/>
-<part name="LED4" library="freetronics-jon" deviceset="RGBLED" device="SMT"/>
+<part name="LED4" library="freetronics-master-v1" deviceset="FREETRONICS-MASTER-V1_RGBLED" device="SMT"/>
 <part name="RN4" library="resistor-dil" deviceset="4R-N" device="CAY16" value="2K2"/>
 <part name="GND16" library="SparkFun" deviceset="GND" device=""/>
@@
 <part name="R25" library="freetronics-jon" deviceset="RESISTOR" device="0402" value="1M 0402"/>
 <part name="XTL5" library="freetronics-jon" deviceset="CRYSTAL-GND" device="3X2" value="SMD3225-16MHZ 3.2 x 2.5mm crystal"/>
-<part name="LED5" library="freetronics-jon" deviceset="RGBLED" device="SMT"/>
+<part name="LED5" library="freetronics-master-v1" deviceset="FREETRONICS-MASTER-V1_RGBLED" device="SMT"/>
 <part name="RN5" library="resistor-dil" deviceset="4R-N" device="CAY16" value="2K2"/>
 <part name="GND22" library="SparkFun" deviceset="GND" device=""/>
@@
 <part name="R30" library="freetronics-jon" deviceset="RESISTOR" device="0402" value="1M 0402"/>
 <part name="XTL6" library="freetronics-jon" deviceset="CRYSTAL-GND" device="3X2" value="SMD3225-16MHZ 3.2 x 2.5mm crystal"/>
-<part name="LED6" library="freetronics-jon" deviceset="RGBLED" device="SMT"/>
+<part name="LED6" library="freetronics-master-v1" deviceset="FREETRONICS-MASTER-V1_RGBLED" device="SMT"/>
 <part name="RN6" library="resistor-dil" deviceset="4R-N" device="CAY16" value="2K2"/>
 <part name="GND30" library="SparkFun" deviceset="GND" device=""/>
@@
 <part name="R36" library="freetronics-jon" deviceset="RESISTOR" device="0402" value="1M 0402"/>
 <part name="XTL7" library="freetronics-jon" deviceset="CRYSTAL-GND" device="3X2" value="SMD3225-16MHZ 3.2 x 2.5mm crystal"/>
-<part name="LED7" library="freetronics-jon" deviceset="RGBLED" device="SMT"/>
+<part name="LED7" library="freetronics-master-v1" deviceset="FREETRONICS-MASTER-V1_RGBLED" device="SMT"/>
 <part name="RN7" library="resistor-dil" deviceset="4R-N" device="CAY16" value="2K2"/>
 <part name="GND38" library="SparkFun" deviceset="GND" device=""/>
@@
 <part name="R40" library="freetronics-jon" deviceset="RESISTOR" device="0402" value="1M 0402"/>
 <part name="XTL8" library="freetronics-jon" deviceset="CRYSTAL-GND" device="3X2" value="SMD3225-16MHZ 3.2 x 2.5mm crystal"/>
-<part name="LED8" library="freetronics-jon" deviceset="RGBLED" device="SMT"/>
+<part name="LED8" library="freetronics-master-v1" deviceset="FREETRONICS-MASTER-V1_RGBLED" device="SMT"/>
 <part name="RN8" library="resistor-dil" deviceset="4R-N" device="CAY16" value="2K2"/>
 <part name="GND43" library="SparkFun" deviceset="GND" device=""/>
@@
 <part name="R44" library="freetronics-jon" deviceset="RESISTOR" device="0402" value="1M 0402"/>
 <part name="XTL9" library="freetronics-jon" deviceset="CRYSTAL-GND" device="3X2" value="SMD3225-16MHZ 3.2 x 2.5mm crystal"/>
-<part name="LED9" library="freetronics-jon" deviceset="RGBLED" device="SMT"/>
+<part name="LED9" library="freetronics-master-v1" deviceset="FREETRONICS-MASTER-V1_RGBLED" device="SMT"/>
 <part name="RN9" library="resistor-dil" deviceset="4R-N" device="CAY16" value="2K2"/>
 <part name="GND48" library="SparkFun" deviceset="GND" device=""/>
@@
 <part name="R48" library="freetronics-jon" deviceset="RESISTOR" device="0402" value="1M 0402"/>
 <part name="XTL10" library="freetronics-jon" deviceset="CRYSTAL-GND" device="3X2" value="SMD3225-16MHZ 3.2 x 2.5mm crystal"/>
-<part name="LED10" library="freetronics-jon" deviceset="RGBLED" device="SMT"/>
+<part name="LED10" library="freetronics-master-v1" deviceset="FREETRONICS-MASTER-V1_RGBLED" device="SMT"/>
 <part name="RN10" library="resistor-dil" deviceset="4R-N" device="CAY16" value="2K2"/>
 <part name="GND53" library="SparkFun" deviceset="GND" device=""/>
@@
 <part name="R52" library="freetronics-jon" deviceset="RESISTOR" device="0402" value="1M 0402"/>
 <part name="XTL11" library="freetronics-jon" deviceset="CRYSTAL-GND" device="3X2" value="SMD3225-16MHZ 3.2 x 2.5mm crystal"/>
-<part name="LED11" library="freetronics-jon" deviceset="RGBLED" device="SMT"/>
+<part name="LED11" library="freetronics-master-v1" deviceset="FREETRONICS-MASTER-V1_RGBLED" device="SMT"/>
 <part name="RN11" library="resistor-dil" deviceset="4R-N" device="CAY16" value="2K2"/>
 <part name="GND58" library="SparkFun" deviceset="GND" device=""/>
@@
 <part name="R56" library="freetronics-jon" deviceset="RESISTOR" device="0402" value="1M 0402"/>
 <part name="XTL12" library="freetronics-jon" deviceset="CRYSTAL-GND" device="3X2" value="SMD3225-16MHZ 3.2 x 2.5mm crystal"/>
-<part name="LED12" library="freetronics-jon" deviceset="RGBLED" device="SMT"/>
+<part name="LED12" library="freetronics-master-v1" deviceset="FREETRONICS-MASTER-V1_RGBLED" device="SMT"/>
 <part name="RN12" library="resistor-dil" deviceset="4R-N" device="CAY16" value="2K2"/>
 <part name="GND63" library="SparkFun" deviceset="GND" device=""/>
@@
 <part name="R61" library="freetronics-jon" deviceset="RESISTOR" device="0402" value="1M 0402"/>
 <part name="XTL13" library="freetronics-jon" deviceset="CRYSTAL-GND" device="3X2" value="SMD3225-16MHZ 3.2 x 2.5mm crystal"/>
-<part name="LED13" library="freetronics-jon" deviceset="RGBLED" device="SMT"/>
+<part name="LED13" library="freetronics-master-v1" deviceset="FREETRONICS-MASTER-V1_RGBLED" device="SMT"/>
 <part name="RN13" library="resistor-dil" deviceset="4R-N" device="CAY16" value="2K2"/>
 <part name="GND68" library="SparkFun" deviceset="GND" device=""/>
@@
 <part name="R65" library="freetronics-jon" deviceset="RESISTOR" device="0402" value="1M 0402"/>
 <part name="XTL14" library="freetronics-jon" deviceset="CRYSTAL-GND" device="3X2" value="SMD3225-16MHZ 3.2 x 2.5mm crystal"/>
-<part name="LED14" library="freetronics-jon" deviceset="RGBLED" device="SMT"/>
+<part name="LED14" library="freetronics-master-v1" deviceset="FREETRONICS-MASTER-V1_RGBLED" device="SMT"/>
 <part name="RN14" library="resistor-dil" deviceset="4R-N" device="CAY16" value="2K2"/>
 <part name="GND79" library="SparkFun" deviceset="GND" device=""/>
@@
 <part name="R69" library="freetronics-jon" deviceset="RESISTOR" device="0402" value="1M 0402"/>
 <part name="XTL15" library="freetronics-jon" deviceset="CRYSTAL-GND" device="3X2" value="SMD3225-16MHZ 3.2 x 2.5mm crystal"/>
-<part name="LED15" library="freetronics-jon" deviceset="RGBLED" device="SMT"/>
+<part name="LED15" library="freetronics-master-v1" deviceset="FREETRONICS-MASTER-V1_RGBLED" device="SMT"/>
 <part name="RN15" library="resistor-dil" deviceset="4R-N" device="CAY16" value="2K2"/>
 <part name="GND89" library="SparkFun" deviceset="GND" device=""/>
@@
 <part name="R73" library="freetronics-jon" deviceset="RESISTOR" device="0402" value="1M 0402"/>
 <part name="XTL16" library="freetronics-jon" deviceset="CRYSTAL-GND" device="3X2" value="SMD3225-16MHZ 3.2 x 2.5mm crystal"/>
-<part name="LED16" library="freetronics-jon" deviceset="RGBLED" device="SMT"/>
+<part name="LED16" library="freetronics-master-v1" deviceset="FREETRONICS-MASTER-V1_RGBLED" device="SMT"/>
 <part name="RN16" library="resistor-dil" deviceset="4R-N" device="CAY16" value="2K2"/>
 <part name="GND96" library="SparkFun" deviceset="GND" device=""/>
