File: ArduSatPayloadProcessorModule.sch (EAGLE design)
At the start: 338 parts, among them IC1 ATMEGA328P QFN32, IC10 ATMEGA328P QFN32, IC11 ATMEGA328P QFN32, IC12 ATMEGA328P QFN32, IC13 ATMEGA328P QFN32, IC14 ATMEGA328P QFN32, IC15 ATMEGA328P QFN32, IC16 ATMEGA328P QFN32, IC17 TXB0104, IC18 TMP102, IC19 TMP102, IC2 ATMEGA328P QFN32, IC20 ATMEGA2561-16MU, IC21 MAX4372F, IC22 MAX4372F, IC23 MUX-74HC4067-QFNSMT, IC24 MUX-74HC4067-QFNSMT, IC3 ATMEGA328P QFN32, IC4 ATMEGA328P QFN32, IC5 ATMEGA328P QFN32, IC6 ATMEGA328P QFN32, IC7 ATMEGA328P QFN32, IC8 ATMEGA328P QFN32, IC9 ATMEGA328P QFN32, P1 microSD, Q1 RJU003N03 N-MOSFET, Q10 RJU003N03 N-MOSFET, Q11 RJU003N03 N-MOSFET, Q12 RJU003N03 N-MOSFET, Q13 RJU003N03 N-MOSFET, Q14 RJU003N03 N-MOSFET, Q15 RJU003N03 N-MOSFET, Q16 RJU003N03 N-MOSFET, Q17 RJU003N03 N-MOSFET, Q18 RJU003N03 N-MOSFET, Q19 RJU003N03 N-MOSFET, Q2 RJU003N03 N-MOSFET, Q20 RJU003N03 N-MOSFET, Q21 RJU003N03 N-MOSFET, Q22 RJU003N03 N-MOSFET, Q23 RJU003N03 N-MOSFET, Q24 RJU003N03 N-MOSFET, Q25 RJU003N03 N-MOSFET, Q26 RJU003N03 N-MOSFET, Q27 RJU003N03 N-MOSFET, Q28 RJU003N03 N-MOSFET, Q29 RJU003N03 N-MOSFET, Q3 RJU003N03 N-MOSFET, Q30 RJU003N03 N-MOSFET, Q31 RJU003N03 N-MOSFET, Q32 RJU003N03 N-MOSFET, Q33 RJU003N03 N-MOSFET, Q34 RJU003N03 N-MOSFET, Q35 RJU003N03 N-MOSFET, Q36 RJU003N03 N-MOSFET, Q37 RJU003N03 N-MOSFET, Q38 RJU003N03 N-MOSFET, Q39 RJU003N03 N-MOSFET, Q4 RJU003N03 N-MOSFET, Q40 RJU003N03 N-MOSFET, Q41 RJU003N03 N-MOSFET, Q42 RJU003N03 N-MOSFET, Q43 RJU003N03 N-MOSFET, Q44 RJU003N03 N-MOSFET, Q45 RJU003N03 N-MOSFET, Q46 RJU003N03 N-MOSFET, Q5 RJU003N03 N-MOSFET, Q6 RJU003N03 N-MOSFET, Q7 RJU003N03 N-MOSFET, Q8 RJU003N03 N-MOSFET, Q9 RJU003N03 N-MOSFET, SW1 ADG801 SOT23-6, SW10 ADG801 SOT23-6, SW11 ADG801 SOT23-6, SW12 ADG801 SOT23-6, SW13 ADG801 SOT23-6, SW14 ADG801 SOT23-6, SW15 ADG801 SOT23-6, SW16 ADG801 SOT23-6, SW17 RESET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

Commit message: Switched PWR LED to 0402
Parts:
- LED17: device freetronics:LED0603 -> freetronics-jon:LED0402
Changed lines of the file:
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@@
 <part name="GND3" library="freetronics-original" deviceset="GND" device=""/>
 <part name="R10" library="freetronics-jon" deviceset="RESISTOR" device="0402" value="2K2 0402"/>
-<part name="LED17" library="freetronics" deviceset="LED" device="0603" value="BLUE 0603"/>
+<part name="LED17" library="freetronics-jon" deviceset="LED" device="0402" value="BLUE 0603"/>
 <part name="U$19" library="SparkFun" deviceset="5V" device=""/>
 <part name="GND23" library="SparkFun" deviceset="GND" device=""/>
